Commit message: Adjusted drone params to be in line with real drone

File: lsy_drone_racing/sim/assets/cf2x.urdf (robot description, URDF)
Before this commit: robot cf2, 6 links, 5 joints
Links:
- link base_link: geometry collision cylinder length=.025 radius=.07; visual mesh filename=./cf2.dae scale=1 1 1
